Commit message: 视觉跟踪优化

File: URDF运动学仿真/urdf/soarmoce_urdf.urdf (robot description, URDF)
Before this commit: robot soarmoce_urdf, 7 links, 6 joints
Joints:
- joint elbow: limit lower=-1.55342947 upper=1.65752103 effort=0 velocity=0 -> lower=-3.14159265 upper=3.14159265 effort=0 velocity=0
- joint shoulder: limit lower=-1.82543714 upper=2.03252454 effort=0 velocity=0 -> lower=-1.57079633 upper=1.57079633 effort=0 velocity=0
- joint shoulder_lift: limit lower=-1.72124222 upper=1.48738250 effort=0 velocity=0 -> lower=-0.78539816 upper=3.14159265 effort=0 velocity=0
- joint wrist: limit lower=-1.59073808 upper=1.52937885 effort=0 velocity=0 -> lower=-1.57079633 upper=1.57079633 effort=0 velocity=0
- joint wrist_roll: limit lower=-3.41464123 upper=0.00920388 effort=0 velocity=0 -> lower=-3.14159265 upper=3.14159265 effort=0 velocity=0

Commit message: Prepare robot arm project for ARM migration

File: URDF运动学仿真/urdf/soarmoce_urdf.urdf (robot description, URDF)
Before this commit: robot soarmoce_urdf, 7 links, 6 joints
Links:
- removed link base
- removed link elbow
- removed link gripper
- removed link shoulder
- removed link shoulder_lift
- removed link wrist
- removed link wrist_roll
- added link Link_1; collision mesh filename=../meshes/Link_1.stl; visual mesh filename=../meshes/Link_1.stl
- added link Link_2; collision mesh filename=../meshes/Link_2.stl; visual mesh filename=../meshes/Link_2.stl
- added link Link_3; collision mesh filename=../meshes/Link_3.stl; visual mesh filename=../meshes/Link_3.stl
- added link Link_4; collision mesh filename=../meshes/Link_4.stl; visual mesh filename=../meshes/Link_4.stl
- added link Link_5; collision mesh filename=../meshes/Link_5.stl; visual mesh filename=../meshes/Link_5.stl
- added link Link_6; collision mesh filename=../meshes/Link_6.stl; visual mesh filename=../meshes/Link_6.stl
- added link base_link; collision mesh filename=../meshes/base_link.stl; visual mesh filename=../meshes/base_link.stl
Joints:
- removed joint elbow
- removed joint gripper
- removed joint shoulder
- removed joint shoulder_lift
- removed joint wrist
- removed joint wrist_roll
- added joint J10: type prismatic, parent base_link, child Link_1, origin xyz=0.13 0.0045 0 rpy=0 -1.57079633 0, axis 0 0 -1, limit lower=-0.1 upper=0.1 effort=100 velocity=0.1
- added joint J11: type revolute, parent Link_1, child Link_2, origin xyz=0.0952507 -0.009787 0.13000505 rpy=0 1.57079633 0, axis 0 0 -1, limit lower=-3.14159 upper=3.14159 effort=10 velocity=1
- added joint J12: type revolute, parent Link_2, child Link_3, origin xyz=-0.030995 3e-8 0.10390639 rpy=1.57079633 0 1.57079633, axis 0 0 -1, limit lower=-3.14159 upper=3.14159 effort=10 velocity=1
- added joint J13: type revolute, parent Link_3, child Link_4, origin xyz=-0.12501147 0.043 -0.002 rpy=3.14159265 0 3.14159265, axis 0 0 1, limit lower=-3.14159 upper=3.14159 effort=10 velocity=1
- added joint J14: type revolute, parent Link_4, child Link_5, origin xyz=-0.00025571 0.1529998 -0.013775 rpy=0 0 0, axis 0 0 -1, limit lower=-3.14159 upper=3.14159 effort=10 velocity=1
- added joint J15: type revolute, parent Link_5, child Link_6, origin xyz=-0.00014171 0.07712488 -0.015925 rpy=-1.57079633 0 -3.13943131, axis 0 0 1, limit lower=-3.14159 upper=3.14159 effort=10 velocity=1
