Commit message: Align URDF geometry and calibration fallback

File: URDF运动学仿真/urdf/soarmoce_urdf.urdf (robot description, URDF)
Before this commit: robot robot, 7 links, 6 joints
Joints:
- joint J10: axis 0 0 -1 -> 0 0 1; origin xyz=0.13 0.0045 0 rpy=0 -1.57079633 0 -> xyz=-0.00000505 -0.005287 0.0922507 rpy=3.14159265 0 3.14159265
- joint J11: axis 0 0 -1 -> 0 0 1; origin xyz=0.0952507 -0.009787 0.13000505 rpy=0 1.57079633 0 -> xyz=0 0 0 rpy=0 0 0
- joint J12: axis 0 0 -1 -> 0 0 1; origin xyz=-0.030995 3e-8 0.10390639 rpy=1.57079633 0 1.57079633 -> xyz=-0.031005 3e-8 -0.10690639 rpy=-1.57079633 0 -1.57079633
- joint J13: axis 0 0 1 -> 0 0 -1; origin xyz=-0.12501147 0.043 -0.002 rpy=3.14159265 0 3.14159265 -> xyz=0.12501147 0.043 0.062 rpy=-3.14159265 0 3.14159265
- joint J14: origin xyz=-0.00025571 0.1529998 -0.013775 rpy=0 0 0 -> xyz=0.153 0.000075 0.011775 rpy=-3.14159265 0 3.14159265
- joint J15: origin xyz=-0.00014171 0.07712488 -0.015925 rpy=-1.57079633 0 -3.13943131 -> xyz=-0.067125 0.00002501 -0.015925 rpy=-1.57079633 0 1.57079618
