Commit message: Update V2 model and synchronize cinematic playback

File: URDF运动学仿真/urdf/v2/soarmoce_urdf.urdf (robot description, URDF)
Before this commit: robot momo_robot_arm_v2, 7 links, 6 joints
Joints:
- joint J10: origin xyz=-0.13 -0.019 -0.022 rpy=1.57079633 0 1.57079633 -> xyz=0.025 0 0 rpy=1.57079633 0 1.57079633
- joint J11: axis 0 0 1 -> 0 0 -1; origin xyz=0.019145 0.107 0.12999495 rpy=0 -1.57079633 -1.57079633 -> xyz=0.000145 0.089 -0.02500505 rpy=0 -1.57079633 -1.57079633
- joint J13: origin xyz=0 0.13000002 -0.0006 rpy=0 0 0 -> xyz=0 0.12999998 -5e-8 rpy=0 0 0
- joint J14: origin xyz=0.14999994 3e-8 -0.05 rpy=0 0 0 -> xyz=0.14999991 3e-8 -0.063 rpy=0 0 0
- joint J15: origin xyz=0.06139999 -0.00439984 0.03045014 rpy=1.57079633 0 -1.57079633 -> xyz=0.06139999 -0.00440002 0.03045014 rpy=1.57079633 0 -1.57079633
